File: e-ink_PCB/_autosave-e-ink_PCB.kicad_pcb (KiCad board)
At the start: 2 copper layers, 71.6 x 33 mm, 10 parts, among them J1 SEEED C3, J3 SHT31, J4 C2, J5 Battery

Commit message: kiCAD shipped
Routing:
- net GND: track 58.1 -> 60.1 mm, vias 17 -> 18
Changed lines of the file:
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@@
 		(tenting front back)
 		(pcbplotparams
-			(layerselection 0x00000000_00000000_55555555_5755f5ff)
+			(layerselection 0x00000000_00000000_55555555_5755557f)
 			(plot_on_all_layers_selection 0x00000000_00000000_00000000_00000000)
 			(disableapertmacros no)
 			(usegerberextensions no)
-			(usegerberattributes yes)
+			(usegerberattributes no)
 			(usegerberadvancedattributes yes)
 			(creategerberjobfile yes)
@@
 			(outputformat 1)
 			(mirror no)
-			(drillshape 1)
+			(drillshape 0)
 			(scaleselection 1)
 			(outputdirectory "")
@@
 		(tags "Through hole pin header THT 1x08 2.54mm single row")
 		(property "Reference" "Display"
-			(at -1.5 20.9 0)
+			(at -3.7 21 0)
 			(layer "F.SilkS")
 			(effects
@@
 		(layer "Edge.Cuts")
 	)
-	(gr_text "+"
-		(at 140.1 108.6 0)
-		(layer "F.Cu")
+	(gr_text "{dblquote}Dreams and Gasoline{dblquote}"
+		(at 121.4 122.5 0)
+		(layer "F.SilkS")
 		(effects
 			(font
-				(size 1.651 1.651)
-				(thickness 0.3302)
-				(bold yes)
+				(size 1.016 1.016)
+				(thickness 0.1524)
 			)
 			(justify left bottom)
 		)
 	)
-	(gr_text "-"
-		(at 142.1 116.8 90)
-		(layer "F.Cu")
+	(gr_text "+"
+		(at 140.1 108.6 0)
+		(layer "F.SilkS")
 		(effects
 			(font
@@
 		)
 	)
-	(gr_text "{dblquote}Dreams and Gasoline{dblquote}"
-		(at 120.1 123.8 0)
+	(gr_text "-"
+		(at 142.1 116.8 90)
 		(layer "F.SilkS")
 		(effects
 			(font
-				(size 1.016 1.016)
-				(thickness 0.1524)
+				(size 1.651 1.651)
+				(thickness 0.3302)
+				(bold yes)
 			)
 			(justify left bottom)
@@
 		(start 76.5 115.66)
 		(end 83.06 115.66)
-		(width 0.2)
+		(width 0.254)
 		(layer "F.Cu")
 		(net 1)
@@
 		(start 104.165 101.5)
 		(end 106.28 101.5)
-		(width 0.2)
+		(width 0.254)
 		(layer "F.Cu")
 		(net 1)
@@
 		(start 88.1 115.8)
 		(end 94.3 109.6)
-		(width 0.2)
+		(width 0.254)
 		(layer "F.Cu")
 		(net 1)
@@
 		(start 83.2 115.8)
 		(end 88.1 115.8)
-		(width 0.2)
+		(width 0.254)
 		(layer "F.Cu")
 		(net 1)
@@
 		(start 102.3 101.5)
 		(end 104.165 101.5)
-		(width 0.2)
+		(width 0.254)
 		(layer "F.Cu")
 		(net 1)
@@
 		(start 106.28 101.5)
 		(end 110.2 97.58)
-		(width 0.2)
+		(width 0.254)
 		(layer "F.Cu")
 		(net 1)
@@
 		(start 97.4 106.4)
 		(end 102.3 101.5)
-		(width 0.2)
+		(width 0.254)
 		(layer "F.Cu")
 		(net 1)
@@
 		(start 94.3 109.6)
 		(end 97.4 106.5)
-		(width 0.2)
+		(width 0.254)
 		(layer "B.Cu")
 		(net 1)
@@
 	)
 	(segment
+		(start 143 112.5)
+		(end 141 112.5)
+		(width 0.2)
+		(layer "F.Cu")
+		(net 16)
+	)
+	(segment
 		(start 120 96.5)
 		(end 126.1 96.5)
@@
 		(net 16)
 	)
+	(via
+		(at 141 112.5)
+		(size 0.6)
+		(drill 0.3)
+		(layers "F.Cu" "B.Cu")
+		(net 16)
+	)
