File: e-ink_PCB_throughole/e-ink_PCB.kicad_pcb (KiCad board)
At the start: 2 copper layers, 71.6 x 33 mm, 10 parts, among them J1 SEEED C3, J3 SHT31, J4 C2, J5 Battery

Commit message: throughole design
Parts:
- J1: footprint Module:XIAO-ESP32C3-SMD_alex -> Module:XIAO-ESP32C3-Throughole_alex
- moved R2 10.2 mm to (101.2, 120.9), turned to 180 degrees
- renumbered Display to J2, MOSFET to Q1
Routing:
- net GND: track 58.1 -> 22.2 mm, vias 17 -> 15
- net Net-(J1-Pin_8): track 34.0 -> 32.8 mm
Other:
- board text added: "Display"

Commit message: updates to KiCAD
Parts:
- J1: value SEEED C3 -> SEED C3
- J4: value C2 -> 100 uF CAP
- J5: value Battery -> Batt Conn
- moved C1 20.3 mm to (83.8, 100.5)
- moved J2 16.2 mm to (76.5, 102.0), turned to 0 degrees
- moved Q1 13.8 mm to (124.1, 115.4)
- moved R1 13.6 mm to (104.5, 116.5)
- moved R2 13.6 mm to (114.8, 120.8)
- moved J4 12.2 mm to (148.0, 98.1)
- moved J5 9.95 mm to (152.9, 111.8)
- moved J3 7.86 mm to (118.1, 97.3)
- moved R3 7.48 mm to (117.7, 109.9)
- moved J1 6.59 mm to (102.6, 103.9)
Connections:
- J1 pad 21: Net-(J2-Pin_3) -> Net-(J2-Pin_8)
- J1 pad 3: Net-(J2-Pin_8) -> Net-(J2-Pin_3)
- J1 pad 4: Net-(J2-Pin_7) -> Net-(J2-Pin_4)
- J1 pad 5: Net-(J2-Pin_6) -> Net-(J2-Pin_5)
- J1 pad 6: Net-(J2-Pin_5) -> Net-(J2-Pin_6)
- J1 pad 7: Net-(J2-Pin_4) -> Net-(J2-Pin_7)
Routing:
- net Net-(J4-Pin_2): track 83.8 -> 3.50 mm
- net Net-(J2-Pin_2): track 41.4 -> 0.20 mm, vias 2 -> 0
- net Net-(J1-Pin_8): track 32.8 -> 4.93 mm, vias 1 -> 0
- net GND: track 22.2 -> 0.00 mm, vias 15 -> 10
- net Net-(J2-Pin_8): track 12.1 -> 0.00 mm
- net Net-(J2-Pin_5): track 12.1 -> 0.00 mm
- net Net-(J2-Pin_3): track 12.1 -> 0.00 mm
- net Net-(J2-Pin_7): track 12.1 -> 0.00 mm
- net Net-(J2-Pin_6): track 12.1 -> 0.10 mm
- net Net-(J2-Pin_4): track 12.1 -> 0.14 mm
- net Net-(Q1-G): track 11.9 -> 0.00 mm
- net Net-(Q1-D): track 9.94 -> 0.00 mm, vias 2 -> 0
- net Net-(J3-Pin_3): track 6.61 -> 0.00 mm
- net Net-(J3-Pin_4): track 6.61 -> 0.00 mm
Other:
- board size 71.6 x 33 mm -> 82.1 x 33 mm
