File: e-ink_PCB_throughole/e-ink_PCB.kicad_sch (KiCad schematic)
At the start: 10 parts, among them J1 SEED C3, J2 e-ink-display, J3 SHT31, J4 100 uF CAP, J5 Batt Conn, Q1 FQP27P06

Commit message: updates to KiCAD
Connections:
- net at J2.BUSY (Pin_8): now also J1.21 (Pin_2); no longer J1.3 (Pin_7)
- net at J2.CS (Pin_7): now also J1.7 (Pin_3); no longer J1.4 (Pin_6)
- net at J2.DC (Pin_6): now also J1.6 (Pin_4); no longer J1.5 (Pin_5)
- net at J2.RES (Pin_5): now also J1.5 (Pin_5); no longer J1.6 (Pin_4)
- net at J2.SCL (Pin_3): now also J1.3 (Pin_7); no longer J1.21 (Pin_2)
- net at J2.SDA (Pin_4): now also J1.4 (Pin_6); no longer J1.7 (Pin_3)
Other:
- moved on the sheet: J2
Changed lines of the file:
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@@
 	(paper "A4")
+	(junction
+		(at 59.69 64.77)
+		(diameter 0)
+		(color 0 0 0 0)
+	)
 	(junction
 		(at 137.16 64.77)
@@
 	)
 	(junction
-		(at 91.44 67.31)
-		(diameter 0)
-		(color 0 0 0 0)
-	)
-	(junction
 		(at 153.67 86.36)
 		(diameter 0)
@@
 	)
 	(junction
-		(at 59.69 66.04)
-		(diameter 0)
-		(color 0 0 0 0)
-	)
-	(junction
 		(at 138.43 95.25)
 		(diameter 0)
@@
 	)
 	(junction
+		(at 100.33 77.47)
+		(diameter 0)
+		(color 0 0 0 0)
+	)
+	(junction
 		(at 153.67 83.82)
 		(diameter 0)
 		(color 0 0 0 0)
 	)
-	(junction
-		(at 59.69 67.31)
-		(diameter 0)
-		(color 0 0 0 0)
-	)
 	(wire
 		(pts
@@
 	(wire
 		(pts
-			(xy 67.31 85.09) (xy 90.17 85.09)
-		)
-		(stroke
-			(width 0)
-			(type default)
-		)
-	)
-	(wire
-		(pts
 			(xy 100.33 80.01) (xy 116.84 80.01)
 		)
@@
 	(wire
 		(pts
+			(xy 100.33 76.2) (xy 91.44 76.2)
+		)
+		(stroke
+			(width 0)
+			(type default)
+		)
+	)
+	(wire
+		(pts
+			(xy 64.77 77.47) (xy 90.17 77.47)
+		)
+		(stroke
+			(width 0)
+			(type default)
+		)
+	)
+	(wire
+		(pts
 			(xy 72.39 72.39) (xy 77.47 72.39)
 		)
@@
 	(wire
 		(pts
-			(xy 67.31 87.63) (xy 90.17 87.63)
+			(xy 62.23 72.39) (xy 64.77 72.39)
+		)
+		(stroke
+			(width 0)
+			(type default)
+		)
+	)
+	(wire
+		(pts
+			(xy 64.77 64.77) (xy 59.69 64.77)
+		)
+		(stroke
+			(width 0)
+			(type default)
+		)
+	)
+	(wire
+		(pts
+			(xy 64.77 85.09) (xy 90.17 85.09)
+		)
+		(stroke
+			(width 0)
+			(type default)
+		)
+	)
+	(wire
+		(pts
+			(xy 59.69 64.77) (xy 59.69 67.31)
 		)
 		(stroke
@@
 	(wire
 		(pts
-			(xy 67.31 82.55) (xy 90.17 82.55)
-		)
-		(stroke
-			(width 0)
-			(type default)
-		)
-	)
-	(wire
-		(pts
-			(xy 59.69 67.31) (xy 59.69 92.71)
-		)
-		(stroke
-			(width 0)
-			(type default)
-		)
-	)
-	(wire
-		(pts
-			(xy 67.31 92.71) (xy 59.69 92.71)
-		)
-		(stroke
-			(width 0)
-			(type default)
-		)
-	)
-	(wire
-		(pts
-			(xy 67.31 77.47) (xy 90.17 77.47)
+			(xy 100.33 77.47) (xy 100.33 76.2)
 		)
 		(stroke
@@
 	(wire
 		(pts
-			(xy 63.5 69.85) (xy 63.5 66.04)
-		)
-		(stroke
-			(width 0)
-			(type default)
-		)
-	)
-	(wire
-		(pts
 			(xy 153.67 86.36) (xy 165.1 86.36)
 		)
@@
 	(wire
 		(pts
-			(xy 91.44 67.31) (xy 77.47 67.31)
+			(xy 77.47 67.31) (xy 109.22 67.31)
 		)
 		(stroke
@@
 	(wire
 		(pts
-			(xy 67.31 74.93) (xy 90.17 74.93)
-		)
-		(stroke
-			(width 0)
-			(type default)
-		)
-	)
-	(wire
-		(pts
 			(xy 137.16 64.77) (xy 137.16 67.31)
 		)
@@
 	(wire
 		(pts
+			(xy 64.77 80.01) (xy 90.17 80.01)
+		)
+		(stroke
+			(width 0)
+			(type default)
+		)
+	)
+	(wire
+		(pts
 			(xy 130.81 95.25) (xy 138.43 95.25)
 		)
@@
 	(wire
 		(pts
-			(xy 59.69 66.04) (xy 59.69 67.31)
-		)
-		(stroke
-			(width 0)
-			(type default)
-		)
-	)
-	(wire
-		(pts
-			(xy 109.22 67.31) (xy 91.44 67.31)
+			(xy 91.44 90.17) (xy 62.23 90.17)
 		)
 		(stroke
@@
 	(wire
 		(pts
+			(xy 64.77 87.63) (xy 90.17 87.63)
+		)
+		(stroke
+			(width 0)
+			(type default)
+		)
+	)
+	(wire
+		(pts
 			(xy 110.49 69.85) (xy 113.03 69.85)
 		)
@@
 	(wire
 		(pts
+			(xy 91.44 76.2) (xy 91.44 90.17)
+		)
+		(stroke
+			(width 0)
+			(type default)
+		)
+	)
+	(wire
+		(pts
 			(xy 137.16 62.23) (xy 137.16 64.77)
 		)
@@
 	(wire
 		(pts
-			(xy 59.69 57.15) (xy 59.69 66.04)
+			(xy 64.77 69.85) (xy 64.77 64.77)
+		)
+		(stroke
+			(width 0)
+			(type default)
+		)
+	)
+	(wire
+		(pts
+			(xy 59.69 57.15) (xy 59.69 64.77)
 		)
 		(stroke
@@
 	(wire
 		(pts
+			(xy 62.23 90.17) (xy 62.23 72.39)
+		)
+		(stroke
+			(width 0)
+			(type default)
+		)
+	)
+	(wire
+		(pts
 			(xy 153.67 86.36) (xy 153.67 95.25)
 		)
@@
 	(wire
 		(pts
+			(xy 64.77 82.55) (xy 90.17 82.55)
+		)
+		(stroke
+			(width 0)
+			(type default)
+		)
+	)
+	(wire
+		(pts
 			(xy 153.67 80.01) (xy 149.86 80.01)
 		)
@@
 	(wire
 		(pts
-			(xy 91.44 67.31) (xy 91.44 90.17)
-		)
-		(stroke
-			(width 0)
-			(type default)
-		)
-	)
-	(wire
-		(pts
 			(xy 125.73 77.47) (xy 116.84 77.47)
 		)
@@
 	(wire
 		(pts
-			(xy 67.31 80.01) (xy 90.17 80.01)
-		)
-		(stroke
-			(width 0)
-			(type default)
-		)
-	)
-	(wire
-		(pts
-			(xy 91.44 90.17) (xy 67.31 90.17)
+			(xy 64.77 74.93) (xy 90.17 74.93)
 		)
 		(stroke
@@
 		(pts
 			(xy 72.39 67.31) (xy 72.39 72.39)
-		)
-		(stroke
-			(width 0)
-			(type default)
-		)
-	)
-	(wire
-		(pts
-			(xy 63.5 66.04) (xy 59.69 66.04)
 		)
 		(stroke
@@
 	(symbol
 		(lib_id "Connector:Conn_01x09_Socket")
-		(at 62.23 82.55 180)
+		(at 69.85 80.01 0)
 		(unit 1)
 		(exclude_from_sim no)
@@
 		(fields_autoplaced yes)
 		(property "Reference" "J2"
-			(at 62.865 69.85 0)
-			(effects
-				(font
-					(size 1.27 1.27)
-				)
+			(at 71.12 77.4699 0)
+			(effects
+				(font
+					(size 1.27 1.27)
+				)
+				(justify left)
 			)
 		)
 		(property "Value" "e-ink-display"
-			(at 62.865 72.39 0)
-			(effects
-				(font
-					(size 1.27 1.27)
-				)
+			(at 71.12 80.0099 0)
+			(effects
+				(font
+					(size 1.27 1.27)
+				)
+				(justify left)
 			)
 		)
 		(property "Footprint" "Connector_PinHeader_2.54mm:PinHeader_1x08_P2.54mm_Vertical"
-			(at 62.23 82.55 0)
+			(at 69.85 80.01 0)
 			(effects
 				(font
@@
 		)
 		(property "Datasheet" "~"
-			(at 62.23 82.55 0)
+			(at 69.85 80.01 0)
 			(effects
 				(font
@@
 		)
 		(property "Description" "Generic connector, single row, 01x09, script generated"
-			(at 62.23 82.55 0)
-			(effects
-				(font
+			(at 69.85 80.01 0)
+			(effects
+				(font
