File: e-ink-PCBs/Throughole-Basic/e-ink_PCB.kicad_pcb (KiCad board)
At the start: 2 copper layers, 62.3 x 31.8 mm, 12 parts, among them J1 SEED C3, J2 e-ink-display, J3 SHT31, J5 Batt Conn, Q2 MOSFET

Commit message: almost final throughole-basic
Parts:
- moved 68k 10.2 mm to (97.9, 121.1), turned to 0 degrees
Routing:
- net Net-(J1-Pin_8): track 28.3 -> 27.1 mm
- added copper zone on B.Cu, net GND
- added copper zone on F.Cu, net GND
Other:
- board text added: "DENTON.WORKS/E-INK"
Changed lines of the file:
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@@
 	(footprint "Resistor_THT:R_Axial_DIN0207_L6.3mm_D2.5mm_P10.16mm_Horizontal"
 		(layer "F.Cu")
-		(at 108.1 121.79 180)
+		(at 97.9 121.12)
 		(descr "Resistor, Axial_DIN0207 series, Axial, Horizontal, pin pitch=10.16mm, 0.25W = 1/4W, length*diameter=6.3*2.5mm^2, http://cdn-reichelt.de/documents/datenblatt/B400/1_4W%23YAG.pdf")
 		(tags "Resistor Axial_DIN0207 series Axial Horizontal pin pitch 10.16mm 0.25W = 1/4W length 6.3mm diameter 2.5mm")
@@
 		(attr through_hole)
 		(fp_line
-			(start 9.12 0)
-			(end 8.35 0)
+			(start 1.04 0)
+			(end 1.81 0)
 			(stroke
 				(width 0.12)
@@
 		)
 		(fp_line
-			(start 1.04 0)
-			(end 1.81 0)
+			(start 9.12 0)
+			(end 8.35 0)
 			(stroke
 				(width 0.12)
@@
 		)
 		(fp_line
-			(start 10.16 0)
-			(end 8.23 0)
+			(start 0 0)
+			(end 1.93 0)
 			(stroke
 				(width 0.1)
@@
 		)
 		(fp_line
-			(start 0 0)
-			(end 1.93 0)
+			(start 10.16 0)
+			(end 8.23 0)
 			(stroke
 				(width 0.1)
@@
 		)
 		(pad "1" thru_hole circle
-			(at 0 0 180)
+			(at 0 0)
 			(size 1.6 1.6)
 			(drill 0.8)
@@
 		)
 		(pad "2" thru_hole circle
-			(at 10.16 0 180)
+			(at 10.16 0)
 			(size 1.6 1.6)
 			(drill 0.8)
@@
 				(thickness 0.15)
 			)
+		)
+	)
+	(gr_text "DENTON.WORKS/E-INK"
+		(at 118.55 95.4 0)
+		(layer "F.SilkS")
+		(effects
+			(font
+				(size 1.524 1.524)
+				(thickness 0.381)
+				(bold yes)
+			)
+			(justify left bottom)
 		)
 	)
@@
 	)
 	(segment
+		(start 97.93 117.51)
+		(end 97.93 121.09)
+		(width 0.2)
+		(layer "F.Cu")
+		(net 10)
+	)
+	(segment
 		(start 98.05 117.33)
 		(end 97.93 117.21)
@@
 	)
 	(segment
-		(start 97.83 121.71)
-		(end 98.03 121.91)
-		(width 0.2)
-		(layer "F.Cu")
-		(net 10)
-	)
-	(segment
-		(start 98.05 121.81)
-		(end 98.05 117.33)
-		(width 0.2)
-		(layer "F.Cu")
-		(net 10)
-	)
-	(segment
 		(start 95.09 96.33)
 		(end 95.44 96.33)
+		(width 0.2)
+		(layer "F.Cu")
+		(net 10)
+	)
+	(segment
+		(start 97.93 121.09)
+		(end 97.9 121.12)
 		(width 0.2)
 		(layer "F.Cu")
@@
 		(net 18)
 	)
+	(zone
+		(net 13)
+		(net_name "GND")
+		(layers "F.Cu" "B.Cu")
+		(hatch edge 0.5)
+		(connect_pads
+			(clearance 0.5)
+		)
+		(min_thickness 0.25)
+		(filled_areas_thickness no)
+		(fill
+			(thermal_gap 0.5)
+			(thermal_bridge_width 0.5)
+		)
+		(polygon
+			(pts
+				(xy 84.6 92.03) (xy 145.95 92.09) (xy 146.02 123.03) (xy 84.72 122.93)
+			)
+		)
+	)
 	(embedded_fonts no)

Commit message: changes to sensor code
Routing:
- net GND: vias 0 -> 10
Other:
- board size 62.3 x 31.8 mm -> 62.2 x 31.9 mm
Changed lines of the file:
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@@
-		)
-		(fp_line
-			(start -1.77 -1.77)
-			(end -1.77 19.55)
-			(stroke
-				(width 0.05)
-				(type solid)
-			)
-			(layer "F.CrtYd")
-		)
-		(fp_line
-			(start -1.77 19.55)
-			(end 1.77 19.55)
-			(stroke
-				(width 0.05)
-				(type solid)
-			)
-			(layer "F.CrtYd")
-		)
-		(fp_line
-			(start 1.77 -1.77)
-			(end -1.77 -1.77)
-			(stroke
-				(width 0.05)
-				(type solid)
-			)
-			(layer "F.CrtYd")
-		)
-		(fp_line
-			(start 1.77 19.55)
-			(end 1.77 -1.77)
-			(stroke
-				(width 0.05)
-				(type solid)
-			)
-			(layer "F.CrtYd")
 		)
 		(fp_line
@@
 	)
 	(gr_rect
-		(start 84.2 91.68)
-		(end 146.54 123.53)
+		(start 84.58 91.695)
+		(end 146.79 123.545)
 		(stroke
 			(width 0.05)
@@
 		(net 12)
 	)
+	(via
+		(at 105 100)
+		(size 0.6)
+		(drill 0.3)
+		(layers "F.Cu" "B.Cu")
+		(free yes)
+		(net 13)
+	)
+	(via
+		(at 120 110)
+		(size 0.6)
+		(drill 0.3)
+		(layers "F.Cu" "B.Cu")
+		(free yes)
+		(net 13)
+	)
+	(via
+		(at 135 110)
+		(size 0.6)
+		(drill 0.3)
+		(layers "F.Cu" "B.Cu")
+		(free yes)
+		(net 13)
+	)
+	(via
+		(at 130 110)
+		(size 0.6)
+		(drill 0.3)
+		(layers "F.Cu" "B.Cu")
+		(free yes)
+		(net 13)
+	)
+	(via
+		(at 105 105)
+		(size 0.6)
+		(drill 0.3)
+		(layers "F.Cu" "B.Cu")
+		(free yes)
+		(net 13)
+	)
+	(via
+		(at 125 110)
+		(size 0.6)
+		(drill 0.3)
+		(layers "F.Cu" "B.Cu")
+		(free yes)
+		(net 13)
+	)
+	(via
+		(at 95 120)
+		(size 0.6)
+		(drill 0.3)
+		(layers "F.Cu" "B.Cu")
+		(free yes)
+		(net 13)
+	)
+	(via
+		(at 95 115)
+		(size 0.6)
+		(drill 0.3)
+		(layers "F.Cu" "B.Cu")
+		(free yes)
+		(net 13)
+	)
+	(via
+		(at 140 105)
+		(size 0.6)
+		(drill 0.3)
+		(layers "F.Cu" "B.Cu")
+		(free yes)
+		(net 13)
+	)
+	(via
+		(at 140 100)
+		(size 0.6)
+		(drill 0.3)
+		(layers "F.Cu" "B.Cu")
+		(free yes)
+		(net 13)
+	)
 	(segment
 		(start 110.09 101.41)
@@
 		(start 141.62 116.64)
 		(end 137.89 120.37)
-		(width 0.2)
+		(width 0.254)
 		(layer "F.Cu")
 		(net 18)
@@
 		(start 137.89 120.37)
 		(end 132.18 120.37)
-		(width 0.2)
+		(width 0.254)
 		(layer "F.Cu")
 		(net 18)
@@
 		(start 116.3525 120.1575)
 		(end 114.59 121.92)
-		(width 0.2)
+		(width 0.254)
 		(layer "F.Cu")
 		(net 18)
@@
 		(start 98.99 106.51)
 		(end 100.57 106.51)
-		(width 0.2)
+		(width 0.254)
 		(layer "F.Cu")
 		(net 18)
@@
 		(start 100.57 106.51)
 		(end 107.35 113.29)
-		(width 0.2)
+		(width 0.254)
 		(layer "F.Cu")
 		(net 18)
@@
 		(start 132.18 120.37)
 		(end 119.7625 120.37)
-		(width 0.2)
+		(width 0.254)
 		(layer "F.Cu")
 		(net 18)
@@
 		(start 107.35 113.29)
 		(end 114.59 120.53)
-		(width 0.2)
+		(width 0.254)
 		(layer "B.Cu")
 		(net 18)
@@
 		(start 114.59 120.53)
 		(end 114.59 121.92)
-		(width 0.2)
+		(width 0.254)
 		(layer "B.Cu")
 		(net 18)
@@
 		(min_thickness 0.25)
 		(filled_areas_thickness no)
-		(fill
+		(fill yes
 			(thermal_gap 0.5)
 			(thermal_bridge_width 0.5)
@@
 		(polygon
 			(pts
-				(xy 84.6 92.03) (xy 145.95 92.09) (xy 146.02 123.03) (xy 84.72 122.93)
-			)
-		)
+				(xy 84.839612 92.030234) (xy 145.95 92.09) (xy 146.02 123.03) (xy 84.959612 122.930391)
+			)
+		)
