File: e-ink-PCBs/Throughole-RTC/e-ink_PCB.kicad_sch (KiCad schematic)
At the start: 15 parts, among them J1 SEED C3, J2 e-ink-display, J3 SHT31, J4 10 uF CAP, J5 Batt Conn, Q1 FQP27P06, Q2 ZXMP4A16G, U1 MCP7940N-xP, Y1 Crystal

Commit message: changes to sensor code
Parts:
- added J6: SD_CARD, symbol Connector:Conn_01x06_Socket
Connections:
- net GND: now also BTTM_68K.2, C2.1, C3.1, J6.GND (Pin_6)
- net at Q1.1 (G), R3.1: now also J1.8 (Pin_6), Q2.1 (G); no longer J1.20 (Pin_7)
- net at U1.1 (X1): now also C2.2, Y1.1
- net at U1.2 (X2): now also C3.2, Y1.2
- net at U1.3 (VBAT): now also BT1.1 (+)
- net at U1.5 (SDA): now also J1.10 (Pin_4), J3.SDA (Pin_4)
- net at U1.6 (SCL): now also J1.9 (Pin_5), J3.SCL (Pin_3)
- net at U1.8 (VCC): now also J3.VIN (Pin_1), Q2.2 (D)
- net at J1.3 (Pin_7), J2.SCL (Pin_3): now also J6.CLK (Pin_4)
- net at J1.4 (Pin_6), J2.SDA (Pin_4): now also J6.MOSI (Pin_3)
- net at J2.VCC (Pin_2): now also J6.3.3V (Pin_1)
- new net: J1.20 (Pin_7), J6.CS (Pin_2)
Other:
- moved on the sheet: BT1, C2, C3, J3, U1, Y1
